File: pcb/microcontroller.kicad_sch (KiCad schematic)
At the start: 0 parts

Commit message: Create STM32 project, expand ADC and GPIO schematic
Parts:
- added C1: 4u7, symbol Device:C
- added C6, C7, C9: 100n, symbol Device:C
- added IC2: STM32C092FCP6, SOP65P640X120-20N, symbol STM32C092FCP6:STM32C092FCP6
- added J14: Screw_Terminal_01x03, symbol Connector:Screw_Terminal_01x03
- added JP1, JP10, JP11, JP12, JP13, JP14, JP15, JP16, JP17, JP18, JP19, JP2, JP20, JP3, JP4, JP5, JP6, JP7, JP8, JP9: SolderJumper_2_Open, Jumper:SolderJumper-2_P1.3mm_Open_TrianglePad1.0x1.5mm, symbol Jumper:SolderJumper_2_Open
- added R28, R29, R30, R31: 10k, symbol Device:R
- added R32, R33, R34, R35: 220, symbol Device:R
- added R38, R39: 1k, symbol Device:R
Connections:
- new net: J14.3 (Pin_3), R38.2
- new net: IC2.3 (PC15-OSCX_OUT), JP13.2 (B)
- new net: J14.2 (Pin_2), R39.1
- new net: IC2.19 (PA14-BOOT0/PA15), JP2.1 (A)
- new net: IC2.2 (PC14-OSCX_IN), JP12.2 (B)
- new net: IC2.12 (PA5), JP9.1 (A)
- new net: IC2.7 (PA0), JP17.2 (B)
- new net: IC2.13 (PA6), JP8.1 (A)
- new net: IC2.16 (PA11_[PA9]), JP5.1 (A)
- new net: IC2.11 (PA4), JP10.1 (A)
- new net: IC2.18 (PA13), JP3.1 (A)
- new net: IC2.4 (VDD/VDDA), JP14.2 (B)
- new net: IC2.1 (PB7/PB8), JP11.2 (B)
- new net: IC2.14 (PA7), JP7.1 (A)
- new net: IC2.15 (PB0/PB1/PB2/PA8), JP6.1 (A)
- new net: IC2.6 (PF2-NRST), JP16.2 (B)
- new net: IC2.9 (PA2), JP19.2 (B)
- new net: IC2.17 (PA12_[PA10]), JP4.1 (A)
- new net: IC2.5 (VSS/VSSA), JP15.2 (B)
- new net: IC2.10 (PA3), JP20.2 (B)
- new net: IC2.20 (PB3/PB4/PB5/PB6), JP1.1 (A)
- new net: IC2.8 (PA1), JP18.2 (B)
- new net +3V3: C1.1, C6.1, J14.1 (Pin_1), JP14.1 (A)
- new net GND: C1.2, C6.2, C7.2, C9.2, JP15.1 (A), R28.1, R29.1, R30.1, R31.1, R38.1
- new net MCU_ENG_THROTTLE: C9.1, JP10.2 (B), R39.2
- new net MCU_NRST: C7.1, JP16.1 (A)
- new net MCU_SOL_EN_1: JP17.1 (A), R28.2, R32.2
- new net MCU_SOL_EN_2: JP18.1 (A), R29.2, R33.2
- new net MCU_SOL_EN_3: JP19.1 (A), R30.2, R35.2
- new net MCU_SOL_EN_4: JP20.1 (A), R31.2, R34.2
- new net SOL_EN_1: R32.1
- new net SOL_EN_2: R33.1
- new net SOL_EN_3: R35.1
- new net SOL_EN_4: R34.1
- no-connect marks 0 -> 12
Other:
- note added: "Engine Throttle"
- note added: "GPIO (SOL_EN) Pulldowns"
- note added: "Hardware Reset Signal"
- note added: "MCU Power"
- note added: "STM32C092FCP6 (TSSOP-20)"

Commit message: Main PCB nearly done, created resolver PCB, more STM32 work
Parts:
- added D1, D2: D, symbol Device:D
- added J15, J16: Screw_Terminal_01x03, symbol Connector:Screw_Terminal_01x03
- added R36: 220, symbol Device:R
- added R37: 10k, symbol Device:R
- added R49: 4k7, Resistor_SMD:R_0603_1608Metric, symbol Device:R
Connections:
- net +3V3: now also D1.2 (A)
- net GND: now also D2.1 (K), R37.1
- net MCU_NRST: no longer JP16.1 (A)
- net SWCLK: now reaches JP2.2 (B)
- net MCU_RESOLVER_CLK: now reaches JP9.2 (B)
- net MCU_RESOLVER_CLK: now also J16.3 (Pin_3)
- net MCU_RESOLVER_MISO: now reaches JP8.2 (B)
- net MCU_RESOLVER_MISO: now also J16.2 (Pin_2)
- net SWDIO: now reaches JP3.2 (B)
- net MCU_SOL_PWM: now reaches JP11.1 (A)
- net MCU_SOL_PWM: now also R36.2, R37.2
- net MCU_RESOLVER_MOSI: now reaches JP7.2 (B)
- net MCU_RESOLVER_MOSI: now also J16.1 (Pin_1)
- net MCU_RESOLVER_CS: now reaches JP6.2 (B)
- net MCU_RESOLVER_CS: now also J15.3 (Pin_3), R49.2
- new net: D2.2 (A), J15.2 (Pin_2)
- new net: D1.1 (K), J15.1 (Pin_1), R49.1
- new net NRST: JP16.1 (A)
- new net SOL_PWM: R36.1
- no-connect marks 12 -> 5
Other:
- note added: "Including reverse-polarity protection diodes"
- note added: "Resolver Connections"
- note added: "Solenoid Power Modulation"
- moved on the sheet: C9, J14, R28, R29, R30, R31, R32, R33, R34, R35, R38, R39

Commit message: Completed all footprints
Parts:
- removed C6, C7, C9: 100n, symbol Device:C
- removed J14, J15, J16: Screw_Terminal_01x03, symbol Connector:Screw_Terminal_01x03
- added C100, C98, C99: 100n, Capacitor_SMD:C_0603_1608Metric, symbol Device:C
- added J12, J14: Screw_Terminal_01x02, footprints:TB005-762-02BE, symbol Connector:Screw_Terminal_01x02
- added J16, J17, J18: TB005-762-02BE, footprints:TB005-762-02BE, symbol TB005-762-02BE:TB005-762-02BE
- C1: footprint (none) -> Capacitor_SMD:C_0805_2012Metric
- D1, D2: footprint (none) -> Diode_SMD:D_0805_2012Metric
- IC2: footprint SOP65P640X120-20N -> footprints:SOP65P640X120-20N
- R28, R29, R30, R31, R32, R33, R34, R35, R36, R37, R38, R39: footprint (none) -> Resistor_SMD:R_0805_2012Metric
- R49: footprint Resistor_SMD:R_0603_1608Metric -> Resistor_SMD:R_0805_2012Metric
Connections:
- net +3V3: now also C99.1, J14.1 (Pin_1), J14.2 (Pin_2)
- net GND: now also C100.2, C98.2, C99.2
- net MCU_ENG_THROTTLE: now also C100.1
- net MCU_NRST: now also C98.1
- net MCU_RESOLVER_CLK: now also J17.2
- net MCU_RESOLVER_CS: now also J17.1
- net MCU_RESOLVER_MISO: now also J16.2
- net MCU_RESOLVER_MOSI: now also J16.1
- net at R38.2: now also J12.2 (Pin_2)
- net at D2.2 (A): now also J18.2
- net at R39.1: now also J12.1 (Pin_1)
- net at D1.1 (K), R49.1: now also J18.1
Other:
- moved on the sheet: D1, D2, R49

Commit message: Grouped all components
Connections:
- net TRTL_GND: now reaches J12.2 (Pin_2), R38.2
- net RESOLVER_GND: now reaches D2.2 (A), J18.2
- net RESOLVER_3V3: now reaches D1.1 (K), J18.1, R49.1
- net TRTL_ADC: now reaches J12.1 (Pin_1), R39.1
Other:
- moved on the sheet: C100, R38, R39
Changed lines of the file:
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@@
 	)
 	(junction
-		(at 57.15 165.1)
+		(at 50.8 165.1)
 		(diameter 0)
 		(color 0 0 0 0)
@@
 	(wire
 		(pts
-			(xy 69.85 171.45) (xy 69.85 167.64)
+			(xy 63.5 171.45) (xy 63.5 167.64)
 		)
 		(stroke
@@
 	(wire
 		(pts
-			(xy 57.15 179.07) (xy 57.15 181.61)
+			(xy 50.8 179.07) (xy 50.8 181.61)
 		)
 		(stroke
@@
 	(wire
 		(pts
-			(xy 67.31 165.1) (xy 76.2 165.1)
+			(xy 60.96 165.1) (xy 76.2 165.1)
 		)
 		(stroke
@@
 	(wire
 		(pts
-			(xy 57.15 171.45) (xy 57.15 165.1)
+			(xy 50.8 171.45) (xy 50.8 165.1)
 		)
 		(stroke
@@
 	(wire
 		(pts
-			(xy 31.75 165.1) (xy 57.15 165.1)
+			(xy 31.75 165.1) (xy 50.8 165.1)
 		)
 		(stroke
@@
 	(wire
 		(pts
-			(xy 69.85 167.64) (xy 76.2 167.64)
+			(xy 63.5 167.64) (xy 76.2 167.64)
 		)
 		(stroke
@@
 	(wire
 		(pts
-			(xy 69.85 179.07) (xy 69.85 181.61)
+			(xy 63.5 179.07) (xy 63.5 181.61)
 		)
 		(stroke
@@
 	(wire
 		(pts
-			(xy 57.15 165.1) (xy 59.69 165.1)
+			(xy 50.8 165.1) (xy 53.34 165.1)
 		)
 		(stroke
@@
 		)
 	)
+	(label "TRTL_ADC"
+		(at 76.2 165.1 180)
+		(effects
+			(font
+				(size 1.27 1.27)
+			)
+			(justify right bottom)
+		)
+	)
 	(label "MCU_SOL_EN_2"
 		(at 97.79 95.25 180)
@@
 		)
 	)
+	(label "TRTL_GND"
+		(at 76.2 167.64 180)
+		(effects
+			(font
+				(size 1.27 1.27)
+			)
+			(justify right bottom)
+		)
+	)
 	(label "MCU_3V3"
 		(at 114.3 91.44 0)
@@
 		)
 	)
+	(label "RESOLVER_3V3"
+		(at 152.4 129.54 0)
+		(effects
+			(font
+				(size 1.27 1.27)
+			)
+			(justify left bottom)
+		)
+	)
+	(label "RESOLVER_GND"
+		(at 148.59 135.89 180)
+		(effects
+			(font
+				(size 1.27 1.27)
+			)
+			(justify right bottom)
+		)
+	)
 	(label "MCU_RESOLVER_CLK"
 		(at 215.9 59.69 180)
@@
 	(symbol
 		(lib_id "Device:R")
-		(at 69.85 175.26 180)
+		(at 63.5 175.26 180)
 		(unit 1)
 		(body_style 1)
@@
 		(dnp no)
 		(property "Reference" "R38"
-			(at 76.2 175.26 90)
+			(at 69.85 175.26 90)
 			(show_name no)
 			(do_not_autoplace no)
@@
 		)
 		(property "Value" "1k"
-			(at 73.66 175.26 90)
+			(at 67.31 175.26 90)
 			(show_name no)
 			(do_not_autoplace no)
@@
 		)
 		(property "Footprint" "Resistor_SMD:R_0805_2012Metric"
-			(at 71.628 175.26 90)
+			(at 65.278 175.26 90)
 			(hide yes)
 			(show_name no)
@@
 		)
 		(property "Datasheet" ""
-			(at 69.85 175.26 0)
+			(at 63.5 175.26 0)
 			(hide yes)
 			(show_name no)
@@
 		)
 		(property "Description" "Resistor"
-			(at 69.85 175.26 0)
+			(at 63.5 175.26 0)
 			(hide yes)
 			(show_name no)
@@
 	(symbol
 		(lib_id "Device:C")
-		(at 57.15 175.26 0)
+		(at 50.8 175.26 0)
 		(unit 1)
 		(body_style 1)
@@
 		(fields_autoplaced yes)
 		(property "Reference" "C100"
-			(at 60.96 173.9899 0)
+			(at 54.61 173.9899 0)
 			(show_name no)
 			(do_not_autoplace no)
@@
 		)
 		(property "Value" "100n"
-			(at 60.96 176.5299 0)
+			(at 54.61 176.5299 0)
 			(show_name no)
 			(do_not_autoplace no)
@@
 		)
 		(property "Footprint" "Capacitor_SMD:C_0603_1608Metric"
-			(at 58.1152 179.07 0)
+			(at 51.7652 179.07 0)
 			(hide yes)
 			(show_name no)
@@
 		)
 		(property "Datasheet" ""
-			(at 57.15 175.26 0)
+			(at 50.8 175.26 0)
 			(hide yes)
 			(show_name no)
@@
 		)
 		(property "Description" "Unpolarized capacitor"
-			(at 57.15 175.26 0)
+			(at 50.8 175.26 0)
 			(hide yes)
 			(show_name no)
@@
 	(symbol
 		(lib_id "power:GND")
-		(at 57.15 181.61 0)
+		(at 50.8 181.61 0)
 		(unit 1)
 		(body_style 1)
@@
 		(fields_autoplaced yes)
 		(property "Reference" "#PWR045"
-			(at 57.15 187.96 0)
+			(at 50.8 187.96 0)
 			(hide yes)
 			(show_name no)
@@
 		)
 		(property "Value" "GND"
-			(at 57.15 186.69 0)
+			(at 50.8 186.69 0)
 			(show_name no)
 			(do_not_autoplace no)
@@
 		)
 		(property "Footprint" ""
-			(at 57.15 181.61 0)
+			(at 50.8 181.61 0)
 			(hide yes)
 			(show_name no)
@@
 		)
 		(property "Datasheet" ""
-			(at 57.15 181.61 0)
+			(at 50.8 181.61 0)
 			(hide yes)
 			(show_name no)
@@
 		)
 		(property "Description" "Power symbol creates a global label with name \"GND\" , ground"
-			(at 57.15 181.61 0)
+			(at 50.8 181.61 0)
 			(hide yes)
 			(show_name no)
@@
 	(symbol
 		(lib_id "power:GND")
-		(at 69.85 181.61 0)
+		(at 63.5 181.61 0)
 		(unit 1)
 		(body_style 1)
@@
 		(fields_autoplaced yes)
 		(property "Reference" "#PWR044"
-			(at 69.85 187.96 0)
+			(at 63.5 187.96 0)
 			(hide yes)
 			(show_name no)
@@
 		)
 		(property "Value" "GND"
-			(at 69.85 186.69 0)
+			(at 63.5 186.69 0)
 			(show_name no)
 			(do_not_autoplace no)
@@
 		)
 		(property "Footprint" ""
-			(at 69.85 181.61 0)
+			(at 63.5 181.61 0)
 			(hide yes)
 			(show_name no)
@@
 		)
 		(property "Datasheet" ""
-			(at 69.85 181.61 0)
+			(at 63.5 181.61 0)
 			(hide yes)
 			(show_name no)
@@
 		)
 		(property "Description" "Power symbol creates a global label with name \"GND\" , ground"
-			(at 69.85 181.61 0)
+			(at 63.5 181.61 0)
 			(hide yes)
 			(show_name no)
@@
 	(symbol
 		(lib_id "Device:R")
-		(at 63.5 165.1 270)
+		(at 57.15 165.1 270)
 		(unit 1)
 		(body_style 1)
@@
 		(fields_autoplaced yes)
 		(property "Reference" "R39"
-			(at 63.5 158.75 90)
+			(at 57.15 158.75 90)
 			(show_name no)
 			(do_not_autoplace no)
@@
 		)
 		(property "Value" "1k"
-			(at 63.5 161.29 90)
+			(at 57.15 161.29 90)
 			(show_name no)
 			(do_not_autoplace no)
@@
 		)
 		(property "Footprint" "Resistor_SMD:R_0805_2012Metric"
-			(at 63.5 163.322 90)
+			(at 57.15 163.322 90)
 			(hide yes)
 			(show_name no)
@@
 		)
 		(property "Datasheet" ""
-			(at 63.5 165.1 0)
+			(at 57.15 165.1 0)
 			(hide yes)
 			(show_name no)
@@
 		)
 		(property "Description" "Resistor"
-			(at 63.5 165.1 0)
+			(at 57.15 165.1 0)
 			(hide yes)
 			(show_name no)
@@
 	)
 	(group ""
-		(members "01310d0c-0be7-4581-8e7a-fa44f0a58582" "13237ecd-e205-4217-9c67-7a5360b6feb8"
-			"142a0709-1e30-43d1-b6ff-ad79be63d8a1" "22a04be5-7be1-4ed2-b2b9-a01202669ddf"
-			"339754b7-e9a7-4de0-b132-e6319d4a5575" "35a3af85-e08c-4ebb-8f78-64e5ae74ceca"
+		(members "01310d0c-0be7-4581-8e7a-fa44f0a58582" "06a5e68e-a61a-4bc8-a65f-5e8e0a8667e3"
+			"13237ecd-e205-4217-9c67-7a5360b6feb8" "142a0709-1e30-43d1-b6ff-ad79be63d8a1"
+			"22a04be5-7be1-4ed2-b2b9-a01202669ddf" "339754b7-e9a7-4de0-b132-e6319d4a5575"
+			"35a3af85-e08c-4ebb-8f78-64e5ae74ceca" "371940f4-f31b-42f4-85cd-2e84826aeeed"
 			"38ecf66b-253a-44d9-bc15-94ec86236dd7" "429d2c7b-dce7-4d63-9fc1-653d814613dd"
 			"4597d9e1-71f8-43b3-8bd7-03110cd71611" "4f15dc06-f658-4cf0-9893-342cb640ad22"
@@
 			"99755573-372a-4bf4-bbe9-70f8d5cae5eb" "9de9c953-9921-4bc0-89e5-11c1aea76108"
 			"a20b02bf-427b-42e1-8b5c-25ce0cc1d0f4" "aa0e3c80-c455-4f61-872d-efba63cf4335"
-			"ba373486-b71c-4b0c-a2bb-df3ba7e68970" "c0367c2e-76fc-4e26-a638-c9f37f7ace18"
-			"c200ce6c-eddd-49dc-b0a2-37cae9731078" "eeb7dbbd-51ce-4473-aa70-996332ae5047"
+			"aa1e7087-8985-4f13-b3b3-07916c455841" "ba373486-b71c-4b0c-a2bb-df3ba7e68970"
+			"c200ce6c-eddd-49dc-b0a2-37cae9731078" "ec09514c-84d7-4110-a5a8-632c214ce9a3"
 		)
 	)

Commit message: PCB nearly done
Parts:
- added R40: 220, Resistor_SMD:R_0805_2012Metric, symbol Device:R
- C100, C99: footprint Capacitor_SMD:C_0603_1608Metric -> Capacitor_SMD:C_0805_2012Metric
- R37: value 10k -> 100k
Connections:
- net MCU_NRST is gone; now on net NRST: C98.1
- net RESOLVER_3V3: now also R40.1; no longer D1.1 (K), R49.1
- new net: D1.1 (K), R40.2, R49.1
Other:
- moved on the sheet: D1, R49
