File: pcb/programmer.kicad_sch (KiCad schematic)
At the start: 1 part, among them U41 STLINK-V3MODS

Commit message: Completed all footprints
Parts:
- removed U41: STLINK-V3MODS, AMS_26_Footprints:STLINK_V3MODS, symbol AMS_26_Symbols:STLINK-V3MODS
- added U1: STLINK-V3MODS, footprints:STLINK_V3MODS, symbol stlink-v3mods:STLINK-V3MODS
Connections:
- net +3V3: now also U1.30 (T_VCC)
- net GND: now also U1.24 (GND), U1.26 (GND2), U1.27 (GND3), U1.29 (GND4), U1.5 (GNDDETECT), U1.8 (GND_2)
- net NRST: now also U1.31 (T_NRST)
- net SWCLK: now also U1.13 (T_JCLK/T_SWCLK)
- net SWDIO: now also U1.4 (T_JTMS/T_SWDIO)
