File: pcb/solenoid_1.kicad_sch (KiCad schematic)
At the start: 15 parts, among them IC1 TPS2819DBVT, J2 Conn_01x01_Pin, J3 Screw_Terminal_01x02, J4 Conn_01x01_Pin, Q1 CSD18542KCS

Commit message: Create STM32 project, expand ADC and GPIO schematic
Parts:
- removed R9: 100, symbol Device:R
Connections:
- net SOL_EN: now also IC1.3 (IN), R10.1

Commit message: Main PCB nearly done, created resolver PCB, more STM32 work
Changed lines of the file:
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@@
+	)
+	(junction
+		(at 209.55 63.5)
+		(diameter 0)
+		(color 0 0 0 0)
 	)
 	(junction
@@
 	)
 	(junction
+		(at 209.55 38.1)
+		(diameter 0)
+		(color 0 0 0 0)
+	)
+	(junction
 		(at 247.65 63.5)
 		(diameter 0)
@@
 	)
 	(junction
-		(at 209.55 38.1)
-		(diameter 0)
-		(color 0 0 0 0)
-	)
-	(junction
 		(at 44.45 46.99)
 		(diameter 0)
@@
 		(color 0 0 0 0)
 	)
-	(junction
-		(at 209.55 63.5)
-		(diameter 0)
-		(color 0 0 0 0)
-	)
 	(wire
 		(pts
@@
 	(wire
 		(pts
+			(xy 203.2 63.5) (xy 209.55 63.5)
+		)
+		(stroke
+			(width 0)
+			(type default)
+		)
+	)
+	(wire
+		(pts
 			(xy 54.61 63.5) (xy 54.61 44.45)
 		)
@@
 	(wire
 		(pts
+			(xy 203.2 38.1) (xy 209.55 38.1)
+		)
+		(stroke
+			(width 0)
+			(type default)
+		)
+	)
+	(wire
+		(pts
 			(xy 153.67 114.3) (xy 146.05 114.3)
 		)
@@
 	(wire
 		(pts
-			(xy 209.55 69.85) (xy 209.55 63.5)
-		)
-		(stroke
-			(width 0)
-			(type default)
-		)
-	)
-	(wire
-		(pts
 			(xy 38.1 46.99) (xy 44.45 46.99)
 		)
@@
 		(pts
 			(xy 25.4 29.21) (xy 114.3 29.21)
-		)
-		(stroke
-			(width 0)
-			(type default)
-		)
-	)
-	(wire
-		(pts
-			(xy 209.55 31.75) (xy 209.55 38.1)
 		)
 		(stroke
@@
 	)
 	(label "SOL-"
-		(at 209.55 69.85 90)
+		(at 203.2 63.5 0)
 		(effects
 			(font
@@
 	)
 	(label "SOL+"
-		(at 209.55 31.75 270)
+		(at 203.2 38.1 0)
 		(effects
 			(font
 				(size 1.27 1.27)
 			)
-			(justify right bottom)
+			(justify left bottom)
 		)
 	)
@@
 	)
 	(group ""
-		(members "0738f25c-d48d-4e56-aced-f8d547b5b2ea" "20e58f6d-6192-45e7-97ce-fb4481d8fc9e"
-			"3a4b742c-91c0-469e-9895-5c20e9101186" "55e59b71-7cc3-493d-91be-c021ba1a604a"
-			"59ad495e-4d15-4ef3-b0c1-19c04054a3a2" "5e127bcf-d55c-486e-9636-9a97d75a5134"
-			"60056fe1-bfa2-402f-8ed1-ebacd9a6f4cb" "60a9d61a-6614-4ed5-a17b-eab4c3f55340"
-			"69f04b03-fef7-40a0-bc34-562216d6f3d2" "6a9973c5-a169-4b9b-8468-cce1f2198a9e"
-			"6c8be35e-de77-47b5-b36a-265b4a9aeba5" "6e7420fe-db0a-4c11-aef5-e94df4b19f74"
-			"6f40bdd6-8014-41d0-9dfb-017f2008049f" "7332bfd5-49de-4611-a2e0-9190bf6cc160"
-			"77fcb79d-9f2b-4782-a546-0d2f557ad044" "797699ea-2005-4498-8c55-54cd85aec307"
-			"824d1d3f-5680-4a9f-a2c7-13cd532a724a" "8f54b4c5-91fb-4425-a8bc-22a915c6d1de"
+		(members "0738f25c-d48d-4e56-aced-f8d547b5b2ea" "088888c1-f323-426b-87e1-3bfde45f146f"
+			"135c6a43-3f59-47c7-9bf9-1e32d8cd0ed0" "20e58f6d-6192-45e7-97ce-fb4481d8fc9e"
+			"3a4b742c-91c0-469e-9895-5c20e9101186" "43fe27f3-b616-407c-b6fc-015631ca73a4"
+			"55e59b71-7cc3-493d-91be-c021ba1a604a" "59ad495e-4d15-4ef3-b0c1-19c04054a3a2"
+			"5e127bcf-d55c-486e-9636-9a97d75a5134" "60056fe1-bfa2-402f-8ed1-ebacd9a6f4cb"
+			"60a9d61a-6614-4ed5-a17b-eab4c3f55340" "69f04b03-fef7-40a0-bc34-562216d6f3d2"
+			"6a9973c5-a169-4b9b-8468-cce1f2198a9e" "6c8be35e-de77-47b5-b36a-265b4a9aeba5"
+			"6e7420fe-db0a-4c11-aef5-e94df4b19f74" "6f40bdd6-8014-41d0-9dfb-017f2008049f"
+			"7332bfd5-49de-4611-a2e0-9190bf6cc160" "77fcb79d-9f2b-4782-a546-0d2f557ad044"
+			"797699ea-2005-4498-8c55-54cd85aec307" "824d1d3f-5680-4a9f-a2c7-13cd532a724a"
+			"8adceec8-eb45-4129-810a-82b5db88528f" "8f54b4c5-91fb-4425-a8bc-22a915c6d1de"
 			"8fb3c8d1-05e5-40eb-bcf4-0db929fd58de" "922b57c4-fa6a-42ce-81fc-37b9bda4baf6"
 			"928b7351-df22-4f10-99eb-9bffee07e496" "973a1369-d79e-4290-b29a-feb079b29811"
 			"976b59c4-2dca-44a8-970c-b2a9af111876" "9a8f15e5-63d2-4c93-a104-5acde1bcb69a"
 			"9bd98cd1-3b21-4366-8ca7-bcf3870ea888" "a0932be2-e51a-4513-8661-c447ff019249"
-			"a1f47dd9-b8e6-4456-825c-d9b40e820953" "b0766375-172c-4f77-ba65-eab9f1de0da5"
-			"c220516d-689a-4a46-b348-2117925a6171" "ce80e19a-343c-48bb-859e-f73e0246a150"
-			"d4772298-75d1-4576-89c2-ccb8e8d09734" "d53095e9-924a-4097-8a2d-14739efa4e66"
-			"d6935c49-fd08-4fed-b77d-e60bc0b901d5" "d72cdc89-df23-40da-86b4-38efcb345f0a"
-			"db111453-e8a8-4bf0-9642-30ab6dcc379e" "e4033601-db7a-4940-97d9-c8bcefa56940"
-			"e8a25e02-082b-4082-98f7-635cb0671171" "f3206449-68d5-47ca-8e29-6185f931a11b"
-			"faa0678a-11fa-43f5-ba29-04073390ac30" "fad6de0d-894d-4cf2-83e6-c6dfaa9d8cb0"
-		)
-	)
+			"ce80e19a-343c-48bb-859e-f73e0246a150" "d4772298-75d1-4576-89c2-ccb8e8d09734"
+			"d53095e9-924a-4097-8a2d-14739efa4e66" "d6935c49-fd08-4fed-b77d-e60bc0b901d5"
+			"d72cdc89-df23-40da-86b4-38efcb345f0a" "db111453-e8a8-4bf0-9642-30ab6dcc379e"
+			"e4033601-db7a-4940-97d9-c8bcefa56940" "e8a25e02-082b-4082-98f7-635cb0671171"
+			"f3206449-68d5-47ca-8e29-6185f931a11b" "faa0678a-11fa-43f5-ba29-04073390ac30"
+		)
+	)

Commit message: Started iteration 4B of CAD today so I have the dimensions of the PCB - have now started layout
Parts:
- renumbered 100n to 100n5, 220u to 220u5
Changed lines of the file:
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@@
 		(in_pos_files yes)
 		(dnp no)
-		(property "Reference" "220u"
+		(property "Reference" "220u5"
 			(at 218.44 49.5299 0)
 			(show_name no)
@@
 				)
 				(path "/8f70d105-0009-40db-8e47-cace6f06f216/9d80248c-e3f3-4348-ae7a-471f00b28847/896e96b4-c651-4615-ba74-5107dc3955e0"
-					(reference "220u")
+					(reference "220u5")
 					(unit 1)
 				)
@@
 		(in_pos_files yes)
 		(dnp no)
-		(property "Reference" "100n"
+		(property "Reference" "100n5"
 			(at 231.14 49.5299 0)
 			(show_name no)
@@
 				)
 				(path "/8f70d105-0009-40db-8e47-cace6f06f216/9d80248c-e3f3-4348-ae7a-471f00b28847/896e96b4-c651-4615-ba74-5107dc3955e0"
-					(reference "100n")
-					(unit 1)
-				)
+					(reference "100n5")
+					(unit 1)
+				)

Commit message: Completed all footprints
Parts:
- removed 100n5, 220u5: C, symbol Device:C
- removed C2: 100n, symbol Device:C
- removed D4: D_TVS, symbol Device:D_TVS
- removed J2, J4: Conn_01x01_Pin, symbol Connector:Conn_01x01_Pin
- added C101, C105: 100n, Capacitor_SMD:C_0805_2012Metric, symbol Device:C
- added C121, C124: 4u7, Capacitor_SMD:C_0805_2012Metric, symbol Device:C
- added D3: SMC30J18A, footprints:DIOM8059X265N, symbol SMC30J18A:SMC30J18A
- D5: footprint (none) -> Diode_SMD:D_0805_2012Metric
- IC1: footprint SOT95P280X145-5N -> footprints:SOT95P280X145-5N
- J3: footprint (none) -> footprints:TB005-762-02BE
- Q1: footprint TO254P470X1016X2016-3P -> footprints:TO254P470X1016X2016-3P
- R10, R5, R7, R8: footprint (none) -> Resistor_SMD:R_0805_2012Metric
Connections:
- net +12V: now also C101.1
- net GND: now also C101.2
- net SOL-: now also C105.2, C121.2, C124.2, D3.2 (A)
- net SOL_PWR: now also C105.1, C121.1, C124.1, D3.1 (K)
Other:
- note added: "TVS diode goes UP from SOL- to SOL+ because it becomes reverse biased at ~18v to clamp voltage transients to ~50v."
- moved on the sheet: J3

Commit message: PCB ready for review
Parts:
- removed Q1: CSD18542KCS, footprints:TO254P470X1016X2016-3P, symbol CSD18542KCS:CSD18542KCS
- added Q1: STH315N10F7-2, footprints:STH315N10F72, symbol STH315N10F7-2:STH315N10F7-2
Connections:
- net GND: now also Q1.3 (S)
- net SOL-: now also Q1.2 (D)
- net at R5.2: now also Q1.1 (G)
Changed lines of the file:
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@@
+	)
+	(symbol
+		(lib_id "STH315N10F7-2:STH315N10F7-2")
+		(at 138.43 129.54 0)
+		(unit 1)
+		(body_style 1)
+		(exclude_from_sim no)
+		(in_bom yes)
+		(on_board yes)
+		(in_pos_files yes)
+		(dnp no)
+		(fields_autoplaced yes)
+		(property "Reference" "Q1"
+			(at 149.86 125.7299 0)
+			(show_name no)
+			(do_not_autoplace no)
+			(effects
+				(font
+					(size 1.27 1.27)
+				)
+				(justify left)
+			)
+		)
+		(property "Value" "STH315N10F7-2"
+			(at 149.86 128.2699 0)
+			(show_name no)
+			(do_not_autoplace no)
+			(effects
+				(font
+					(size 1.27 1.27)
+				)
+				(justify left)
+			)
+		)
+		(property "Footprint" "footprints:STH315N10F72"
+			(at 149.86 228.27 0)
+			(hide yes)
+			(show_name no)
+			(do_not_autoplace no)
+			(effects
+				(font
+					(size 1.27 1.27)
+				)
+				(justify left top)
+			)
+		)
+		(property "Datasheet" "https://www.st.com/resource/en/datasheet/sth315n10f7-2.pdf"
+			(at 149.86 328.27 0)
+			(hide yes)
+			(show_name no)
+			(do_not_autoplace no)
+			(effects
+				(font
+					(size 1.27 1.27)
+				)
+				(justify left top)
+			)
+		)
+		(property "Description" "Automotive-grade N-channel 100 V, 2.1 m typ., 180 A STripFET F7 Power MOSFETs in an HPAK2 and HPAK6 packages"
+			(at 138.43 129.54 0)
+			(hide yes)
+			(show_name no)
+			(do_not_autoplace no)
+			(effects
+				(font
+					(size 1.27 1.27)
+				)
+			)
+		)
+		(property "Height" "4.9"
+			(at 149.86 528.27 0)
+			(hide yes)
+			(show_name no)
+			(do_not_autoplace no)
+			(effects
+				(font
+					(size 1.27 1.27)
+				)
+				(justify left top)
+			)
+		)
+		(property "Mouser Part Number" "511-STH315N10F7-2"
+			(at 149.86 628.27 0)
+			(hide yes)
+			(show_name no)
+			(do_not_autoplace no)
+			(effects
+				(font
+					(size 1.27 1.27)
+				)
+				(justify left top)
+			)
+		)
+		(property "Mouser Price/Stock" "https://www.mouser.co.uk/ProductDetail/STMicroelectronics/STH315N10F7-2?qs=DqCdCwOw4%2F6biN%2FHDRW73g%3D%3D"
+			(at 149.86 728.27 0)
+			(hide yes)
+			(show_name no)
+			(do_not_autoplace no)
+			(effects
+				(font
+					(size 1.27 1.27)
+				)
+				(justify left top)
+			)
+		)
+		(property "Manufacturer_Name" "STMicroelectronics"
+			(at 149.86 828.27 0)
+			(hide yes)
+			(show_name no)
+			(do_not_autoplace no)
+			(effects
+				(font
+					(size 1.27 1.27)
+				)
+				(justify left top)
+			)
+		)
+		(property "Manufacturer_Part_Number" "STH315N10F7-2"
+			(at 149.86 928.27 0)
+			(hide yes)
+			(show_name no)
+			(do_not_autoplace no)
+			(effects
+				(font
+					(size 1.27 1.27)
+				)
+				(justify left top)
+			)
+		)
+		(pin "1"
+		)
+		(pin "2"
+		)
+		(pin "3"
+		)
+		(instances
+			(project "SolenoidEngine4"
+				(path "/8f70d105-0009-40db-8e47-cace6f06f216/9d80248c-e3f3-4348-ae7a-471f00b28847/1e189177-1ffd-48bf-8381-80b2ae3aeecb"
+					(reference "Q4")
+					(unit 1)
+				)
+				(path "/8f70d105-0009-40db-8e47-cace6f06f216/9d80248c-e3f3-4348-ae7a-471f00b28847/5e7b7f5b-7602-483d-9622-47b5c34c6ce4"
+					(reference "Q2")
+					(unit 1)
+				)
+				(path "/8f70d105-0009-40db-8e47-cace6f06f216/9d80248c-e3f3-4348-ae7a-471f00b28847/896e96b4-c651-4615-ba74-5107dc3955e0"
+					(reference "Q1")
+					(unit 1)
+				)
+				(path "/8f70d105-0009-40db-8e47-cace6f06f216/9d80248c-e3f3-4348-ae7a-471f00b28847/dcd1f385-6e3d-442d-bc05-0404acb533c3"
+					(reference "Q3")
+					(unit 1)
+				)
+			)
+		)
 	)
 	(symbol
@@
 				(path "/8f70d105-0009-40db-8e47-cace6f06f216/9d80248c-e3f3-4348-ae7a-471f00b28847/dcd1f385-6e3d-442d-bc05-0404acb533c3"
 					(reference "D6")
-					(unit 1)
-				)
-			)
-		)
-	)
-	(symbol
-		(lib_id "CSD18542KCS:CSD18542KCS")
-		(at 138.43 129.54 0)
-		(unit 1)
-		(body_style 1)
-		(exclude_from_sim no)
-		(in_bom yes)
-		(on_board yes)
-		(in_pos_files yes)
-		(dnp no)
-		(fields_autoplaced yes)
-		(property "Reference" "Q1"
-			(at 149.86 125.7299 0)
-			(show_name no)
-			(do_not_autoplace no)
-			(effects
-				(font
-					(size 1.27 1.27)
-				)
-				(justify left)
-			)
-		)
-		(property "Value" "CSD18542KCS"
-			(at 149.86 128.2699 0)
-			(show_name no)
-			(do_not_autoplace no)
-			(effects
-				(font
-					(size 1.27 1.27)
-				)
-				(justify left)
-			)
-		)
-		(property "Footprint" "footprints:TO254P470X1016X2016-3P"
-			(at 149.86 228.27 0)
-			(hide yes)
-			(show_name no)
-			(do_not_autoplace no)
-			(effects
-				(font
-					(size 1.27 1.27)
-				)
-				(justify left top)
-			)
-		)
-		(property "Datasheet" "http://www.ti.com/lit/gpn/csd18542kcs"
-			(at 149.86 328.27 0)
-			(hide yes)
-			(show_name no)
-			(do_not_autoplace no)
-			(effects
-				(font
-					(size 1.27 1.27)
-				)
-				(justify left top)
-			)
-		)
-		(property "Description" "CSD18542KCS 60-V N-Channel NexFET&#153; Power MOSFET"
-			(at 138.43 129.54 0)
-			(hide yes)
-			(show_name no)
-			(do_not_autoplace no)
-			(effects
-				(font
-					(size 1.27 1.27)
-				)
-			)
-		)
-		(property "Height" "4.7"
-			(at 149.86 528.27 0)
-			(hide yes)
-			(show_name no)
-			(do_not_autoplace no)
-			(effects
-				(font
-					(size 1.27 1.27)
-				)
-				(justify left top)
-			)
-		)
-		(property "Mouser Part Number" "595-CSD18542KCS"
-			(at 149.86 628.27 0)
-			(hide yes)
-			(show_name no)
-			(do_not_autoplace no)
-			(effects
-				(font
-					(size 1.27 1.27)
-				)
-				(justify left top)
-			)
-		)
-		(property "Mouser Price/Stock" "https://www.mouser.co.uk/ProductDetail/Texas-Instruments/CSD18542KCS?qs=sICFeol8QWE7Rbjncdrc5g%3D%3D"
-			(at 149.86 728.27 0)
-			(hide yes)
-			(show_name no)
-			(do_not_autoplace no)
-			(effects
-				(font
-					(size 1.27 1.27)
-				)
-				(justify left top)
-			)
-		)
-		(property "Manufacturer_Name" "Texas Instruments"
-			(at 149.86 828.27 0)
-			(hide yes)
-			(show_name no)
-			(do_not_autoplace no)
-			(effects
-				(font
-					(size 1.27 1.27)
-				)
-				(justify left top)
-			)
-		)
-		(property "Manufacturer_Part_Number" "CSD18542KCS"
-			(at 149.86 928.27 0)
-			(hide yes)
-			(show_name no)
-			(do_not_autoplace no)
-			(effects
-				(font
-					(size 1.27 1.27)
-				)
-				(justify left top)
-			)
-		)
-		(pin "3"
-		)
-		(pin "1"
-		)
-		(pin "2"
-		)
-		(instances
-			(project "SolenoidEngine4"
-				(path "/8f70d105-0009-40db-8e47-cace6f06f216/9d80248c-e3f3-4348-ae7a-471f00b28847/1e189177-1ffd-48bf-8381-80b2ae3aeecb"
-					(reference "Q4")
-					(unit 1)
-				)
-				(path "/8f70d105-0009-40db-8e47-cace6f06f216/9d80248c-e3f3-4348-ae7a-471f00b28847/5e7b7f5b-7602-483d-9622-47b5c34c6ce4"
-					(reference "Q2")
-					(unit 1)
-				)
-				(path "/8f70d105-0009-40db-8e47-cace6f06f216/9d80248c-e3f3-4348-ae7a-471f00b28847/896e96b4-c651-4615-ba74-5107dc3955e0"
-					(reference "Q1")
-					(unit 1)
-				)
-				(path "/8f70d105-0009-40db-8e47-cace6f06f216/9d80248c-e3f3-4348-ae7a-471f00b28847/dcd1f385-6e3d-442d-bc05-0404acb533c3"
-					(reference "Q3")
 					(unit 1)
 				)
@@
 			"95e72fad-54db-417d-bcf1-211183cd4500" "ba42f1a9-0794-4faa-ab2c-77a4a763f0dd"
 			"c8868067-eb68-4cd9-856c-0ecee558d5bf" "ca700e9d-3273-43aa-a7d5-1623a6594ace"
-			"d40a2724-6a23-4e16-9d88-1cfe834c42fe" "d51c5b2c-0304-48b8-90d2-0ea5a588fdc6"
-			"de6f766e-5547-40c5-a4b4-ba799aab76e4" "e3db0938-7360-425a-a375-e89cef00c7fd"
+			"d15dada4-0a1c-484f-8708-17cf576c9279" "d40a2724-6a23-4e16-9d88-1cfe834c42fe"
+			"d51c5b2c-0304-48b8-90d2-0ea5a588fdc6" "de6f766e-5547-40c5-a4b4-ba799aab76e4"
 			"e969f6b6-75ae-4887-9943-c92048c50cc6" "f83bff44-db5c-435b-9e28-0bb8f10d1607"
 		)
