File: pcb/SolenoidEngine4.kicad_pcb (KiCad board)
At the start: 2 copper layers, 7.7 x 7.7 mm, 1 part

Commit message: Started iteration 4B of CAD today so I have the dimensions of the PCB - have now started layout
Parts:
- added C117: 10u, Capacitor_SMD:C_0603_1608Metric, F.Cu at (66.2, 72.0)
- added C119: 4u7, Capacitor_SMD:C_0805_2012Metric, F.Cu at (63.7, 78.5)
- added C120: 1u, Capacitor_SMD:C_0805_2012Metric, F.Cu at (63.7, 81.5)
- added D17: LED, LED_SMD:LED_0603_1608Metric, F.Cu at (72.2, 81.0)
- added IC1: TPS2819DBVT, footprints:SOT95P280X145-5N, F.Cu at (70.5, 103.4)
- added IC2: STM32C092FCP6, footprints:SOP65P640X120-20N, F.Cu at (90.0, 130.0)
- added IC3: TPS2819DBVT, footprints:SOT95P280X145-5N, F.Cu at (84.5, 103.4)
- added IC4: TPS2819DBVT, footprints:SOT95P280X145-5N, F.Cu at (98.7, 103.4)
- added IC5: TPS2819DBVT, footprints:SOT95P280X145-5N, F.Cu at (112.5, 103.4)
- added IC6: TPS2819DBVT, footprints:SOT95P280X145-5N, F.Cu at (97.4, 80.2)
- added IC7: LDL1117S33R, footprints:SOT230P700X180-4N, F.Cu at (90.0, 76.0)
- added JP1: SolderJumper_2_Open, Jumper:SolderJumper-2_P1.3mm_Open_TrianglePad1.0x1.5mm, F.Cu at (84.0, 122.0)
- added JP10: SolderJumper_2_Open, Jumper:SolderJumper-2_P1.3mm_Open_TrianglePad1.0x1.5mm, F.Cu at (100.7, 136.0)
- added JP11: SolderJumper_2_Open, Jumper:SolderJumper-2_P1.3mm_Open_TrianglePad1.0x1.5mm, F.Cu at (79.3, 124.0)
- added JP12: SolderJumper_2_Open, Jumper:SolderJumper-2_P1.3mm_Open_TrianglePad1.0x1.5mm, F.Cu at (79.3, 127.0)
- added JP13: SolderJumper_2_Open, Jumper:SolderJumper-2_P1.3mm_Open_TrianglePad1.0x1.5mm, F.Cu at (79.3, 130.0)
- added JP14: SolderJumper_2_Open, Jumper:SolderJumper-2_P1.3mm_Open_TrianglePad1.0x1.5mm, F.Cu at (79.3, 133.0)
- added JP15: SolderJumper_2_Open, Jumper:SolderJumper-2_P1.3mm_Open_TrianglePad1.0x1.5mm, F.Cu at (79.3, 136.0)
- added JP16: SolderJumper_2_Open, Jumper:SolderJumper-2_P1.3mm_Open_TrianglePad1.0x1.5mm, F.Cu at (84.0, 138.0)
- added JP17: SolderJumper_2_Open, Jumper:SolderJumper-2_P1.3mm_Open_TrianglePad1.0x1.5mm, F.Cu at (87.0, 138.0)
- added JP18: SolderJumper_2_Open, Jumper:SolderJumper-2_P1.3mm_Open_TrianglePad1.0x1.5mm, F.Cu at (90.0, 138.0)
- added JP19: SolderJumper_2_Open, Jumper:SolderJumper-2_P1.3mm_Open_TrianglePad1.0x1.5mm, F.Cu at (93.0, 138.0)
- added JP2: SolderJumper_2_Open, Jumper:SolderJumper-2_P1.3mm_Open_TrianglePad1.0x1.5mm, F.Cu at (87.0, 122.0)
- added JP20: SolderJumper_2_Open, Jumper:SolderJumper-2_P1.3mm_Open_TrianglePad1.0x1.5mm, F.Cu at (96.0, 138.0)
- added JP3: SolderJumper_2_Open, Jumper:SolderJumper-2_P1.3mm_Open_TrianglePad1.0x1.5mm, F.Cu at (90.0, 122.0)
- added JP4: SolderJumper_2_Open, Jumper:SolderJumper-2_P1.3mm_Open_TrianglePad1.0x1.5mm, F.Cu at (93.0, 122.0)
- added JP5: SolderJumper_2_Open, Jumper:SolderJumper-2_P1.3mm_Open_TrianglePad1.0x1.5mm, F.Cu at (96.0, 122.0)
- added JP6: SolderJumper_2_Open, Jumper:SolderJumper-2_P1.3mm_Open_TrianglePad1.0x1.5mm, F.Cu at (100.7, 124.0)
- added JP7: SolderJumper_2_Open, Jumper:SolderJumper-2_P1.3mm_Open_TrianglePad1.0x1.5mm, F.Cu at (100.7, 127.0)
- added JP8: SolderJumper_2_Open, Jumper:SolderJumper-2_P1.3mm_Open_TrianglePad1.0x1.5mm, F.Cu at (100.7, 130.0)
- added JP9: SolderJumper_2_Open, Jumper:SolderJumper-2_P1.3mm_Open_TrianglePad1.0x1.5mm, F.Cu at (100.7, 133.0)
- added Q1: CSD18542KCS, footprints:TO254P470X1016X2016-3P, F.Cu at (71.5, 98.9)
- added Q2: CSD18542KCS, footprints:TO254P470X1016X2016-3P, F.Cu at (85.5, 98.9)
- added Q3: CSD18542KCS, footprints:TO254P470X1016X2016-3P, F.Cu at (99.7, 98.9)
- added Q4: CSD18542KCS, footprints:TO254P470X1016X2016-3P, F.Cu at (113.5, 98.9)
- added Q5: CSD18542KCS, footprints:TO254P470X1016X2016-3P, F.Cu at (111.5, 83.9)
- added R113: 4k7, Resistor_SMD:R_0603_1608Metric, F.Cu at (66.2, 74.5)
- added R49: 4k7, Resistor_SMD:R_0603_1608Metric, F.Cu at (114.0, 119.0)
- added REF**: M8_Ground, SolenoidEngine4:M8_Ground, F.Cu at (50.0, 180.0)
- added REF**: M8_Ground, SolenoidEngine4:M8_Ground, F.Cu at (50.0, 50.0)
- added REF**: M8_Ground, SolenoidEngine4:M8_Ground, F.Cu at (140.0, 180.0)
- added REF**: M8_Ground, SolenoidEngine4:M8_Ground, F.Cu at (140.0, 50.0)
- moved REF** 98.3 mm to (106.9, 29.1)
Routing:
- net (no net): track 0.00 -> 56.6 mm
- net Net-(IC2-PA2): track 0.00 -> 11.0 mm
- net Net-(IC2-PA14-BOOT0/PA15): track 0.00 -> 11.0 mm
- net Net-(IC2-PB3/PB4/PB5/PB6): track 0.00 -> 10.7 mm
- net Net-(IC2-PA3): track 0.00 -> 10.7 mm
- net Net-(IC2-VSS/VSSA): track 0.00 -> 10.4 mm
- net Net-(IC2-PB0/PB1/PB2/PA8): track 0.00 -> 10.4 mm
- net Net-(IC2-PA1): track 0.00 -> 9.78 mm
- net Net-(IC2-PA13): track 0.00 -> 9.78 mm
- net Net-(IC2-PF2-NRST): track 0.00 -> 9.22 mm
- net Net-(IC2-PA11_[PA9]): track 0.00 -> 9.22 mm
- net Net-(IC2-PA0): track 0.00 -> 9.10 mm
- net Net-(IC2-PA12_[PA10]): track 0.00 -> 9.10 mm
- net Net-(IC2-VDD/VDDA): track 0.00 -> 8.71 mm
- net Net-(IC2-PA7): track 0.00 -> 8.71 mm
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- added copper zone on B.Cu, net (none)
- added copper zone on F.Cu, net (none)
Other:
- board size 7.7 x 7.7 mm -> 118 x 158 mm
- board text added: "3V3"
- board text added: "ADC_TRTL"
- board text added: "GND"
- board text added: "NRST"
- board text added: "RES_CLK"
- board text added: "RES_CS"
- board text added: "RES_MISO"
- board text added: "RES_MOSI"
- board text added: "Rear Back"
- board text added: "SOL_1"
- board text added: "SOL_2"
- board text added: "SOL_3"
- board text added: "SOL_4"
- board text added: "SOL_PWM"
- board text added: "ST Microelectronics NV"
- board text added: "STM32C092FCP6"
- board text added: "SWCLK"
- board text added: "SWDIO"
- board text added: "x"

Commit message: Completed all footprints
Parts:
- added 100n1: C5, Capacitor_SMD:C_0805_2012Metric, F.Cu at (209.3, 75.7)
- added 220u1: C4, Capacitor_SMD:CP_Elec_10x10, F.Cu at (200.3, 80.1)
- added C1: 4u7, Capacitor_SMD:C_0805_2012Metric, F.Cu at (188.5, 71.8)
- added C100: 100n, Capacitor_SMD:C_0603_1608Metric, F.Cu at (179.8, 76.6)
- added C101: 100n, Capacitor_SMD:C_0805_2012Metric, F.Cu at (195.2, 103.5)
- added C102: 100n, Capacitor_SMD:C_0805_2012Metric, F.Cu at (206.1, 89.5)
- added C103: 100n, Capacitor_SMD:C_0805_2012Metric, F.Cu at (206.1, 103.5)
- added C104: 100n, Capacitor_SMD:C_0805_2012Metric, F.Cu at (195.2, 89.5)
- added C105: 100n, Capacitor_SMD:C_0805_2012Metric, F.Cu at (195.2, 106.6)
- added C106: 100n, Capacitor_SMD:C_0805_2012Metric, F.Cu at (206.1, 92.5)
- added C107: 100n, Capacitor_SMD:C_0805_2012Metric, F.Cu at (206.1, 106.6)
- added C108: 100n, Capacitor_SMD:C_0805_2012Metric, F.Cu at (195.2, 92.5)
- added C109: 100n, Capacitor_SMD:C_0805_2012Metric, F.Cu at (209.3, 78.7)
- added C121: 4u7, Capacitor_SMD:C_0805_2012Metric, F.Cu at (195.2, 109.6)
- added C122: 4u7, Capacitor_SMD:C_0805_2012Metric, F.Cu at (206.1, 95.5)
- added C123: 4u7, Capacitor_SMD:C_0805_2012Metric, F.Cu at (206.1, 109.6)
- added C124: 4u7, Capacitor_SMD:C_0805_2012Metric, F.Cu at (195.2, 112.6)
- added C125: 4u7, Capacitor_SMD:C_0805_2012Metric, F.Cu at (206.1, 98.5)
- added C126: 4u7, Capacitor_SMD:C_0805_2012Metric, F.Cu at (206.1, 112.6)
- added C127: 4u7, Capacitor_SMD:C_0805_2012Metric, F.Cu at (195.2, 95.5)
- added C128: 4u7, Capacitor_SMD:C_0805_2012Metric, F.Cu at (195.2, 98.5)
- added C98: 100n, Capacitor_SMD:C_0603_1608Metric, F.Cu at (179.8, 71.6)
- added C99: 100n, Capacitor_SMD:C_0603_1608Metric, F.Cu at (179.8, 74.1)
- added D1: D, Diode_SMD:D_0805_2012Metric, F.Cu at (184.0, 71.8)
- added D11: LED, Diode_SMD:D_0805_2012Metric, F.Cu at (199.7, 98.4)
- added D2: D, Diode_SMD:D_0805_2012Metric, F.Cu at (184.0, 74.9)
- added D3: SMC30J18A, footprints:DIOM8059X265N, F.Cu at (225.8, 98.2)
- added D4: SMC30J18A, footprints:DIOM8059X265N, F.Cu at (238.6, 85.4)
- added D5: LED, Diode_SMD:D_0805_2012Metric, F.Cu at (199.7, 112.4)
- added D6: SMC30J18A, footprints:DIOM8059X265N, F.Cu at (238.6, 98.2)
- added D7: LED, Diode_SMD:D_0805_2012Metric, F.Cu at (210.6, 98.4)
- added D8: SMC30J18A, footprints:DIOM8059X265N, F.Cu at (225.8, 85.4)
- added D9: LED, Diode_SMD:D_0805_2012Metric, F.Cu at (210.6, 112.4)
- added J15: TB005-762-02BE, footprints:TB005-762-02BE, F.Cu at (198.4, 64.7)
- added J16: TB005-762-02BE, footprints:TB005-762-02BE, F.Cu at (164.8, 64.7)
- added J17: TB005-762-02BE, footprints:TB005-762-02BE, F.Cu at (164.8, 80.4)
- added J18: TB005-762-02BE, footprints:TB005-762-02BE, F.Cu at (164.8, 96.0)
- added R10: 100k, Resistor_SMD:R_0805_2012Metric, F.Cu at (199.7, 109.4)
- added R12: 100k, Resistor_SMD:R_0805_2012Metric, F.Cu at (210.6, 92.4)
- added R13: 100k, Resistor_SMD:R_0805_2012Metric, F.Cu at (210.6, 95.4)
- added R14: 1k, Resistor_SMD:R_0805_2012Metric, F.Cu at (235.4, 90.8)
- added R16: 100k, Resistor_SMD:R_0805_2012Metric, F.Cu at (210.6, 103.5)
- added R17: 100k, Resistor_SMD:R_0805_2012Metric, F.Cu at (210.6, 106.5)
- added R18: 10, Resistor_SMD:R_0805_2012Metric, F.Cu at (210.6, 109.4)
- added R19: 1k, Resistor_SMD:R_0805_2012Metric, F.Cu at (235.4, 103.5)
- added R21: 100k, Resistor_SMD:R_0805_2012Metric, F.Cu at (199.7, 89.5)
- added R22: 100k, Resistor_SMD:R_0805_2012Metric, F.Cu at (199.7, 92.4)
- added R23: 10, Resistor_SMD:R_0805_2012Metric, F.Cu at (199.7, 95.4)
- added R24: 1k, Resistor_SMD:R_0805_2012Metric, F.Cu at (222.7, 90.8)
- added R25: 100k, Resistor_SMD:R_0805_2012Metric, F.Cu at (213.5, 60.0)
- added R26: 100k, Resistor_SMD:R_0805_2012Metric, F.Cu at (235.4, 108.5)
- added R27: 10, Resistor_SMD:R_0805_2012Metric, F.Cu at (213.5, 62.9)
- added R28: 10k, Resistor_SMD:R_0805_2012Metric, F.Cu at (180.0, 60.0)
- added R29: 10k, Resistor_SMD:R_0805_2012Metric, F.Cu at (180.0, 62.9)
- added R30: 10k, Resistor_SMD:R_0805_2012Metric, F.Cu at (180.0, 65.9)
- added R31: 10k, Resistor_SMD:R_0805_2012Metric, F.Cu at (180.0, 68.8)
- added R32: 220, Resistor_SMD:R_0805_2012Metric, F.Cu at (184.4, 60.0)
- added R33: 220, Resistor_SMD:R_0805_2012Metric, F.Cu at (184.4, 62.9)
- added R34: 220, Resistor_SMD:R_0805_2012Metric, F.Cu at (184.4, 65.9)
- added R35: 220, Resistor_SMD:R_0805_2012Metric, F.Cu at (184.4, 68.8)
- added R36: 220, Resistor_SMD:R_0805_2012Metric, F.Cu at (188.8, 60.0)
- added R37: 10k, Resistor_SMD:R_0805_2012Metric, F.Cu at (188.8, 62.9)
- added R38: 1k, Resistor_SMD:R_0805_2012Metric, F.Cu at (188.8, 65.9)
- added R39: 1k, Resistor_SMD:R_0805_2012Metric, F.Cu at (188.8, 68.8)
- added R5: 10, Resistor_SMD:R_0805_2012Metric, F.Cu at (199.7, 103.5)
- added R6: 10, Resistor_SMD:R_0805_2012Metric, F.Cu at (210.6, 89.5)
- added R7: 100k, Resistor_SMD:R_0805_2012Metric, F.Cu at (199.7, 106.5)
- added R8: 1k, Resistor_SMD:R_0805_2012Metric, F.Cu at (222.7, 103.5)
- C117: value 10u -> 220u; footprint Capacitor_SMD:C_0603_1608Metric -> Capacitor_SMD:C_0805_2012Metric
- C119, C120: moved to B.Cu
- D17: footprint LED_SMD:LED_0603_1608Metric -> Diode_SMD:D_0805_2012Metric
- R113, R49: footprint Resistor_SMD:R_0603_1608Metric -> Resistor_SMD:R_0805_2012Metric
- moved C119 27.4 mm to (91.0, 76.0), turned to 90 degrees
- moved C120 21.0 mm to (84.0, 76.0), turned to 90 degrees

Commit message: Grouped all components
Parts:
- removed the REF** at (50.0, 180.0)
- removed the REF** at (50.0, 50.0)
- removed the REF** at (140.0, 180.0)
- removed the REF** at (140.0, 50.0)
- added J10: Screw_Terminal_01x02, footprints:TB005-762-02BE, F.Cu at (376.4, 91.0)
- added J12: Screw_Terminal_01x02, footprints:TB005-762-02BE, F.Cu at (55.2, 308.8)
- added J13: Screw_Terminal_01x02, footprints:TB005-762-02BE, F.Cu at (396.4, 91.0)
- added J14: Screw_Terminal_01x02, footprints:TB005-762-02BE, F.Cu at (55.2, 324.4)
- added J3: Screw_Terminal_01x02, footprints:TB005-762-02BE, F.Cu at (336.4, 91.0)
- added J7: Screw_Terminal_01x02, footprints:TB005-762-02BE, F.Cu at (356.4, 91.0)
- added U1: STLINK-V3MODS, footprints:STLINK_V3MODS, F.Cu at (127.6, 354.6)
- moved IC5 303.5 mm to (415.8, 117.0)
- moved Q4 284.6 mm to (397.9, 107.0)
- moved IC4 281.6 mm to (379.8, 121.0)
- moved IC3 277.7 mm to (361.8, 120.0)
- moved Q3 275.9 mm to (375.5, 105.9)
- moved IC1 272.9 mm to (343.0, 118.0)
- moved Q2 272.1 mm to (357.5, 105.9)
- moved Q1 265.6 mm to (336.9, 107.0)
- moved J16 260.2 mm to (198.2, 322.8)
- moved J17 260.2 mm to (198.2, 338.4)
- moved C98 244.6 mm to (97.8, 302.0)
- moved R38 235.3 mm to (181.0, 301.0)
- moved J18 231.6 mm to (175.2, 327.4)
- moved R33 229.4 mm to (88.1, 271.1)
- moved R34 229.4 mm to (88.1, 274.1)
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Connections:
- net Net-(D1-K) renamed /Microcontroller/RESOLVER_3V3
- net Net-(D2-A) renamed /Microcontroller/RESOLVER_GND
- R38 pad 2: Net-(J14-Pin_3) -> /Microcontroller/TRTL_GND
- R39 pad 1: Net-(J14-Pin_2) -> /Microcontroller/TRTL_ADC

Commit message: PCB nearly done
Parts:
- added R40: 220, Resistor_SMD:R_0805_2012Metric, F.Cu at (220.0, 118.0)
- added REF**: M8_Ground, SolenoidEngine4:M8_Ground, F.Cu at (50.0, 50.0)
- added REF**: M8_Ground, SolenoidEngine4:M8_Ground, F.Cu at (50.0, 140.0)
- added REF**: M8_Ground, SolenoidEngine4:M8_Ground, F.Cu at (230.0, 50.0)
- added REF**: M8_Ground, SolenoidEngine4:M8_Ground, F.Cu at (230.0, 140.0)
- C100, C99: footprint Capacitor_SMD:C_0603_1608Metric -> Capacitor_SMD:C_0805_2012Metric
- C117: footprint Capacitor_SMD:C_0805_2012Metric -> Capacitor_SMD:CP_Elec_10x10
- C119, C120: moved to F.Cu
- C4: renamed from 220u1; value C4 -> 220u
- C5: renamed from 100n1; value C5 -> 100n
- R37: value 10k -> 100k
- moved R8 261.9 mm to (82.0, 60.0), turned to -90 degrees
- moved D3 259.3 mm to (86.0, 53.0), turned to 90 degrees
- moved D5 258.1 mm to (84.0, 60.0), turned to -90 degrees
- moved U1 256.0 mm to (52.0, 110.0), turned to 90 degrees
- moved R7 253.2 mm to (96.0, 65.1), turned to 90 degrees
- moved C105 251.5 mm to (86.0, 60.0), turned to -90 degrees
- moved C124 249.7 mm to (88.0, 60.0), turned to -90 degrees
- moved IC1 249.7 mm to (99.0, 65.1), turned to -90 degrees
- moved R10 249.1 mm to (97.0, 61.1), turned to 0 degrees
- moved C121 247.6 mm to (90.0, 60.0), turned to -90 degrees
- moved J7 244.8 mm to (116.2, 138.4)
- moved J16 244.8 mm to (228.4, 79.8), turned to 90 degrees
- moved C101 244.2 mm to (101.0, 61.1), turned to 180 degrees
- moved R5 244.1 mm to (103.0, 67.0)
- moved R6 242.3 mm to (117.0, 123.0), turned to 180 degrees
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Connections:
- C98 pad 1: /Microcontroller/MCU_NRST -> /Microcontroller/NRST
- D1 pad 1: /Microcontroller/RESOLVER_3V3 -> Net-(D1-K)
- R49 pad 1: /Microcontroller/RESOLVER_3V3 -> Net-(D1-K)
Routing:
- net /Solenoids/Solenoid 1/SOL+: track 0.00 -> 447.4 mm
- net /Microcontroller/SWDIO: track 0.00 -> 177.3 mm, vias 0 -> 6
- net /Microcontroller/SWCLK: track 0.00 -> 163.7 mm, vias 0 -> 6
- net /Microcontroller/NRST: track 0.00 -> 154.4 mm, vias 0 -> 4
- net /Microcontroller/SOL_PWM: track 0.00 -> 140.5 mm, vias 0 -> 2
- net GND: track 0.00 -> 136.7 mm, vias 0 -> 652
- net /Microcontroller/MCU_ENG_THROTTLE: track 0.00 -> 107.5 mm, vias 0 -> 4
- net /Microcontroller/SOL_EN_1: track 0.00 -> 104.1 mm, vias 0 -> 2
- net /Microcontroller/SOL_EN_2: track 0.00 -> 71.8 mm, vias 0 -> 2
- net /Microcontroller/MCU_RESOLVER_MISO: track 0.00 -> 63.8 mm
- net (no net): track 56.6 -> 0.00 mm
- net /Microcontroller/SOL_EN_3: track 0.00 -> 53.3 mm, vias 0 -> 3
- net /Microcontroller/MCU_RESOLVER_CLK: track 0.00 -> 50.2 mm
- net /Microcontroller/MCU_RESOLVER_MOSI: track 0.00 -> 49.2 mm, vias 0 -> 1
- net /Solenoids/Solenoid 3/SOL-: track 0.00 -> 48.3 mm, vias 0 -> 5
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- added copper zone on In2.Cu, net +12V
- added copper zone on In1.Cu, net +3V3
- added copper zone on B.Cu, net GND
- added copper zone on F.Cu, net GND
- removed copper zone on B.Cu, net (none)
- removed copper zone on F.Cu, net (none)
Other:
- board size 118 x 158 mm -> 208 x 118 mm
- copper layers 2 -> 4
- board text added: "12V POWER"
- board text added: "R3V3"
- board text added: "RCLK"
- board text added: "RECS"
- board text added: "RGND"
- board text added: "RMISO"
- board text added: "RMOSI"
- board text added: "SL1-"
- board text added: "SL2-"
- board text added: "SL3-"
- board text added: "SL4-"
- board text added: "SOL+"
- board text added: "T3V3"
- board text added: "TADC"
- board text added: "TGND"
- board text added: "USB+"
- board text added: "USB-"

Commit message: PCB ready for review
Parts:
- Q1, Q2, Q3, Q4, Q5: value CSD18542KCS -> STH315N10F7-2; footprint footprints:TO254P470X1016X2016-3P -> footprints:STH315N10F72
- moved Q1 11.2 mm to (113.0, 66.0), turned to 0 degrees
- moved Q3 11.1 mm to (173.0, 66.4), turned to 0 degrees
- moved Q4 11.1 mm to (167.0, 123.6), turned to 180 degrees
- moved Q2 11.1 mm to (107.0, 123.6), turned to 180 degrees
- moved Q5 9.79 mm to (79.0, 82.4)
- moved R38 5.00 mm to (97.0, 130.0)
- moved C100 4.00 mm to (94.0, 126.0)
- moved R39 4.00 mm to (94.0, 130.0)
- moved REF** 2.00 mm to (30.6, 87.7)
- moved C5 1.41 mm to (88.0, 92.0)
Connections:
- REF** pad 1: (no net) -> GND (x4)
Routing:
- net /Solenoids/Solenoid 1/SOL+: track 447.4 -> 360.2 mm
- net +12V: track 37.0 -> 48.4 mm
- net Net-(Q2-G): track 3.69 -> 10.4 mm
- net Net-(Q4-G): track 3.69 -> 10.4 mm
- net Net-(Q3-G): track 3.69 -> 10.4 mm
- net Net-(Q1-G): track 3.69 -> 9.99 mm
- net GND: track 136.7 -> 142.8 mm, vias 652 -> 598
- net /Microcontroller/MCU_ENG_THROTTLE: track 107.5 -> 111.6 mm
- net /Microcontroller/TRTL_GND: track 8.24 -> 10.3 mm
- net /Solenoids/Solenoid 4/SOL-: track 48.3 -> 50.4 mm, vias 5 -> 6
- net /Solenoids/Solenoid 3/SOL-: track 48.3 -> 50.4 mm, vias 5 -> 6
- net /Solenoids/Solenoid 2/SOL-: track 48.3 -> 50.4 mm, vias 5 -> 6
- net Net-(D7-A): track 0.00 -> 2.01 mm
- net Net-(D11-A): track 0.00 -> 2.01 mm
- net Net-(D9-A): track 0.00 -> 2.01 mm
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
Commit message: Fixed a couple minor issues, re-ran DRC, added my name :)
Other:
- board text added: "Only took me 3 years..."
- board text added: "SOL1+"
- board text added: "SOL1-"
- board text added: "SOL2+"
- board text added: "SOL2-"
- board text added: "SOL3+"
- board text added: "SOL3-"
- board text added: "SOL4+"
- board text added: "SOL4-"
- board text added: "Solenoid Engine #4 Adam Spencer @ atom-dispencer Open-Source on GitHub"
- board text removed: "SL1-"
- board text removed: "SL2-"
- board text removed: "SL3-"
- board text removed: "SL4-"
- board text removed: "SOL+"
Changed lines of the file:
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@@
 		)
 		(embedded_fonts no)
-		(model "STH315N10F7-2.stp"
+		(model "${KIPRJMOD}/lib/3dmodels/STH315N10F7-2.stp"
 			(offset
-				(xyz 0 6.519999883 0)
+				(xyz 0 0 0)
 			)
 			(scale
@@
 			)
 			(rotate
-				(xyz 0 0 0)
+				(xyz -0 -0 -0)
 			)
 		)
@@
 		)
 		(embedded_fonts no)
-		(model "STH315N10F7-2.stp"
+		(model "${KIPRJMOD}/lib/3dmodels/STH315N10F7-2.stp"
 			(offset
-				(xyz 0 6.519999883 0)
+				(xyz 0 0 0)
 			)
 			(scale
@@
 			)
 			(rotate
-				(xyz 0 0 0)
+				(xyz -0 -0 -0)
 			)
 		)
@@
 		)
 		(embedded_fonts no)
-		(model "SMC30J18A.stp"
+		(model "${KIPRJMOD}/lib/3dmodels/SMC30J18A.stp"
 			(offset
 				(xyz 0 0 1.230000001)
@@
 		)
 		(embedded_fonts no)
-		(model "SMC30J18A.stp"
+		(model "${KIPRJMOD}/lib/3dmodels/SMC30J18A.stp"
 			(offset
 				(xyz 0 0 1.230000001)
@@
 		)
 		(embedded_fonts no)
-		(model "STH315N10F7-2.stp"
+		(model "${KIPRJMOD}/lib/3dmodels/STH315N10F7-2.stp"
 			(offset
-				(xyz 0 6.519999883 0)
+				(xyz 0 0 0)
 			)
 			(scale
@@
 			)
 			(rotate
-				(xyz 0 0 0)
+				(xyz -0 -0 -0)
 			)
 		)
@@
 		)
 		(embedded_fonts no)
-		(model "STH315N10F7-2.stp"
+		(model "${KIPRJMOD}/lib/3dmodels/STH315N10F7-2.stp"
 			(offset
-				(xyz 0 6.519999883 0)
+				(xyz 0 0 0)
 			)
 			(scale
@@
 			)
 			(rotate
-				(xyz 0 0 0)
+				(xyz -0 -0 -0)
 			)
 		)
@@
 		)
 		(embedded_fonts no)
-		(model "SMC30J18A.stp"
+		(model "${KIPRJMOD}/lib/3dmodels/SMC30J18A.stp"
 			(offset
 				(xyz 0 0 1.230000001)
@@
 		)
 		(embedded_fonts no)
-		(model "STH315N10F7-2.stp"
+		(model "${KIPRJMOD}/lib/3dmodels/STH315N10F7-2.stp"
 			(offset
-				(xyz 0 6.519999883 0)
+				(xyz 0 0 0)
 			)
 			(scale
@@
 			)
 			(rotate
-				(xyz 0 0 0)
+				(xyz -0 -0 -0)
 			)
 		)
@@
 		)
 		(embedded_fonts no)
-		(model "SMC30J18A.stp"
+		(model "${KIPRJMOD}/lib/3dmodels/SMC30J18A.stp"
 			(offset
 				(xyz 0 0 1.230000001)
@@
 		)
 		(embedded_fonts no)
-		(model "TB005-762-02BE.stp"
+		(model "${KIPRJMOD}/lib/3dmodels/TB005-762-02BE.stp"
 			(offset
 				(xyz 7.550000077 -7.899999977 0)
@@
 		)
 	)
-	(gr_text "SOL+"
-		(at 115 150 0)
+	(gr_text "SOL2+"
+		(at 114 150 0)
 		(layer "F.SilkS" knockout)
 		(effects
@@
 		)
 	)
-	(gr_text "SL2-"
-		(at 125 150 0)
+	(gr_text "SOL2-"
+		(at 126 150 0)
 		(layer "F.SilkS" knockout)
 		(effects
@@
 		)
 	)
-	(gr_text "SOL+"
-		(at 175 150 0)
+	(gr_text "SOL4+"
+		(at 174 150 0)
 		(layer "F.SilkS" knockout)
 		(effects
@@
 		)
 	)
-	(gr_text "SL4-"
-		(at 185 150 0)
+	(gr_text "SOL4-"
+		(at 186 150 0)
 		(layer "F.SilkS" knockout)
 		(effects
@@
 		)
 	)
-	(gr_text "SL1-"
-		(at 95 40 180)
+	(gr_text "SOL1-"
+		(at 94 40 180)
 		(layer "F.SilkS" knockout)
 		(effects
@@
 		)
 	)
-	(gr_text "SOL+"
-		(at 105 40 180)
+	(gr_text "SOL1+"
+		(at 106 40 180)
 		(layer "F.SilkS" knockout)
 		(effects
@@
 		)
 	)
-	(gr_text "SL3-"
-		(at 155 40 180)
+	(gr_text "SOL3-"
+		(at 154 40 180)
 		(layer "F.SilkS" knockout)
 		(effects
@@
 		)
 	)
-	(gr_text "SOL+"
-		(at 165 40 180)
+	(gr_text "SOL3+"
+		(at 166 40 180)
 		(layer "F.SilkS" knockout)
 		(effects
@@
 		)
 	)
+	(gr_text "Solenoid Engine #4\nAdam Spencer @ atom-dispencer\nOpen-Source on GitHub"
+		(at 140 93 0)
+		(layer "F.SilkS")
+		(effects
+			(font
+				(size 3 2.1)
+				(thickness 0.525)
+				(bold yes)
+			)
+		)
+	)
+	(gr_text "Only took me 3 years..."
+		(at 140 93 0)
+		(layer "B.SilkS")
+		(effects
+			(font
+				(size 3 2.1)
+				(thickness 0.525)
+				(bold yes)
+			)
+			(justify mirror)
+		)
+	)
